Commit message: rxd2

File: ROS/usydrx_sim_bringup/urdf/usyd_vrx_wamv.urdf (robot description, URDF)
Before this commit: robot WAM-V, 15 links, 14 joints
Links:
- added link wamv/front_camera_link, mass 0.3; collision box size=0.036 0.03 0.03; collision cylinder length=0.042 radius=0.015
- added link wamv/front_camera_link_optical
- added link wamv/front_camera_post_arm_link, mass 0.1; collision cylinder length=0.065 radius=0.008; visual mesh filename=package://vrx_gazebo/models/sensor_post/mesh/sensor_post_ar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
- added link wamv/front_camera_post_link, mass 0.06884999999999994; collision cylinder length=0.07649999999999993 radius=0.0076; visual cylinder length=0.07649999999999993 radius=0.0076
- added link wamv/left_camera_link, mass 0.3; collision box size=0.036 0.03 0.03; collision cylinder length=0.042 radius=0.015
- added link wamv/left_camera_link_optical
- added link wamv/left_camera_post_arm_link, mass 0.1; collision cylinder length=0.065 radius=0.008; visual mesh filename=package://vrx_gazebo/models/sensor_post/mesh/sensor_post_ar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
- added link wamv/left_camera_post_link, mass 0.06884999999999994; collision cylinder length=0.07649999999999993 radius=0.0076; visual cylinder length=0.07649999999999993 radius=0.0076
- added link wamv/lidar_wamv_front_link, mass 1; collision cylinder length=0.075 radius=0.055; visual mesh filename=package://vrx_gazebo/models/3d_lidar/mesh/3d_lidar.dae
- added link wamv/lidar_wamv_front_post_arm_link, mass 0.1; collision cylinder length=0.065 radius=0.008; visual mesh filename=package://vrx_gazebo/models/sensor_post/mesh/sensor_post_ar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
- added link wamv/lidar_wamv_front_post_link, mass 0.18315000000000006; collision cylinder length=0.20350000000000007 radius=0.0076; visual cylinder length=0.20350000000000007 radius=0.0076
- added link wamv/right_camera_link, mass 0.3; collision box size=0.036 0.03 0.03; collision cylinder length=0.042 radius=0.015
- added link wamv/right_camera_link_optical
- added link wamv/right_camera_post_arm_link, mass 0.1; collision cylinder length=0.065 radius=0.008; visual mesh filename=package://vrx_gazebo/models/sensor_post/mesh/sensor_post_ar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
- added link wamv/right_camera_post_link, mass 0.06884999999999994; collision cylinder length=0.07649999999999993 radius=0.0076; visual cylinder length=0.07649999999999993 radius=0.0076
Joints:
- added joint wamv/base_to_front_camera_post_joint: type fixed, parent wamv/base_link, child wamv/front_camera_post_link, origin xyz=0.85 0.0 1.3347499999999999 rpy=0 0 0
- added joint wamv/base_to_left_camera_post_joint: type fixed, parent wamv/base_link, child wamv/left_camera_post_link, origin xyz=0.7999999999999999 -0.1 1.3347499999999999 rpy=0 0 0
- added joint wamv/base_to_lidar_wamv_front_post_joint: type fixed, parent wamv/base_link, child wamv/lidar_wamv_front_post_link, origin xyz=0.78 0.0 1.39825 rpy=0 0 0
- added joint wamv/base_to_right_camera_post_joint: type fixed, parent wamv/base_link, child wamv/right_camera_post_link, origin xyz=0.7999999999999999 0.1 1.3347499999999999 rpy=0 0 0
- added joint wamv/front_camera_post_arm_to_front_camera_joint: type fixed, parent wamv/front_camera_post_arm_link, child wamv/front_camera_link, origin xyz=0.02 0 0.027 rpy=0 0.0 0.0
- added joint wamv/front_camera_post_to_front_camera_post_arm_joint: type fixed, parent wamv/front_camera_post_link, child wamv/front_camera_post_arm_link, origin xyz=0.03 0 0.038250000000000034 rpy=0 0 0
- added joint wamv/front_camera_to_front_camera_link_optical_joint: type fixed, parent wamv/front_camera_link, child wamv/front_camera_link_optical, origin xyz=0 0 0 rpy=-1.5707963267948966 0 -1.5707963267948966
- added joint wamv/left_camera_post_arm_to_left_camera_joint: type fixed, parent wamv/left_camera_post_arm_link, child wamv/left_camera_link, origin xyz=0.02 0 0.027 rpy=0 0.0 -1.0471975511965976
- added joint wamv/left_camera_post_to_left_camera_post_arm_joint: type fixed, parent wamv/left_camera_post_link, child wamv/left_camera_post_arm_link, origin xyz=0.03 0 0.038250000000000034 rpy=0 0 0
- added joint wamv/left_camera_to_left_camera_link_optical_joint: type fixed, parent wamv/left_camera_link, child wamv/left_camera_link_optical, origin xyz=0 0 0 rpy=-1.5707963267948966 0 -1.5707963267948966
- added joint wamv/lidar_wamv_front_post_arm_to_lidar_wamv_front_joint: type fixed, parent wamv/lidar_wamv_front_post_arm_link, child wamv/lidar_wamv_front_link, origin xyz=0.04 0 0.05 rpy=0 0.20943951023931956 0
- added joint wamv/lidar_wamv_front_post_to_lidar_wamv_front_post_arm_joint: type fixed, parent wamv/lidar_wamv_front_post_link, child wamv/lidar_wamv_front_post_arm_link, origin xyz=0.03 0 0.10175000000000005 rpy=0 0 0
- added joint wamv/right_camera_post_arm_to_right_camera_joint: type fixed, parent wamv/right_camera_post_arm_link, child wamv/right_camera_link, origin xyz=0.02 0 0.027 rpy=0 0.0 1.0471975511965976
- added joint wamv/right_camera_post_to_right_camera_post_arm_joint: type fixed, parent wamv/right_camera_post_link, child wamv/right_camera_post_arm_link, origin xyz=0.03 0 0.038250000000000034 rpy=0 0 0
- added joint wamv/right_camera_to_right_camera_link_optical_joint: type fixed, parent wamv/right_camera_link, child wamv/right_camera_link_optical, origin xyz=0 0 0 rpy=-1.5707963267948966 0 -1.5707963267948966

File: ROS/usydrx_sim_bringup/wamv_config/component_config.xacro (robot description, xacro)
@@ -2,8 +2,14 @@
 <robot xmlns:xacro="http://ros.org/wiki/xacro" name="wam-v-components">
   <xacro:macro name="yaml_components">
+    <!-- === wamv_camera === -->
+      <xacro:wamv_camera name="front_camera" x="0.9" y="0" z="1.4" Y="${radians(0)}" P="${radians(0)}" />
+      <xacro:wamv_camera name="right_camera" x="0.85" y="0.1" z="1.4" Y="${radians(60)}" P="${radians(0)}" />
+      <xacro:wamv_camera name="left_camera" x="0.85" y="-0.1" z="1.4" Y="${radians(-60)}" P="${radians(0)}" />
     <!-- === wamv_gps === -->
       <xacro:wamv_gps name="gps_wamv" x="-0.85" />
     <!-- === wamv_imu === -->
       <xacro:wamv_imu name="imu_wamv" y="-0.2" />
+    <!-- === lidar === -->
+      <xacro:lidar name="lidar_wamv_front" type="16_beam" x="0.85" y="0" z="1.55" P="${radians(12)}" />
   </xacro:macro>
 </robot>

Commit message: rxd5

File: ROS/usydrx_sim_bringup/urdf/usyd_vrx_wamv.urdf (robot description, URDF)
Before this commit: robot WAM-V, 30 links, 29 joints
Joints:
- joint wamv/front_camera_post_arm_to_front_camera_joint: origin xyz=0.02 0 0.027 rpy=0 0.0 0.0 -> xyz=0.941 -0.005 1.426 rpy=-0.009 0.189 -0.041; parent wamv/front_camera_post_arm_link -> wamv/base_link
- joint wamv/left_camera_post_arm_to_left_camera_joint: origin xyz=0.02 0 0.027 rpy=0 0.0 -1.0471975511965976 -> xyz=0.892 0.095 1.435 rpy=0.156 0.108 0.979; parent wamv/left_camera_post_arm_link -> wamv/base_link
- joint wamv/right_camera_post_arm_to_right_camera_joint: origin xyz=0.02 0 0.027 rpy=0 0.0 1.0471975511965976 -> xyz=0.878 -0.103 1.438 rpy=-0.171 0.083 -1.117; parent wamv/right_camera_post_arm_link -> wamv/base_link
